File: QL_Miracle_Midi.kicad_pcb (KiCad board)
At the start: 2 copper layers, 131.4 x 105.4 mm, 32 parts, among them J1 QL_cartridge_ROM, J2 DIN-5, J3 DIN-5, J4 DIN-5, U1 Z80CPU, U10 74LS74, U2 6264, U3 74LS374, U4 74LS374, U5 74LS10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

Commit message: pinout of midi update
Parts:
- J2, J3, J4: footprint 8bits:DIN-5-female-pcb-horizontal -> 8bits:DIN-5-MIDI-female-pcb-horizontal
Connections:
- J3 pad 3: unconnected-(J3-Pad3) -> GND
- J4 pad 3: unconnected-(J4-Pad3) -> GND
- U6 pad 23: unconnected-(U6-~{DCD}-Pad23) -> GND
- U6 pad 24: unconnected-(U6-~{CTS}-Pad24) -> GND
Routing:
- net Net-(D1-A): track 30.5 -> 26.2 mm
- net Net-(J3-Pad2): track 15.9 -> 14.4 mm
- net Net-(J4-Pad2): track 15.9 -> 14.4 mm
