File: QL_Miracle_Midi.kicad_sch (KiCad schematic)
At the start: 32 parts, among them J1 QL_cartridge_ROM, J2 DIN-5, J3 DIN-5, J4 DIN-5, U1 Z80CPU, U10 74LS74, U2 6264, U3 74LS374, U4 74LS374, U5 74LS10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

Commit message: pinout of midi update
Parts:
- J2, J3, J4: footprint 8bits:DIN-5-female-pcb-horizontal -> 8bits:DIN-5-MIDI-female-pcb-horizontal
Connections:
- net GND: now also J3.3, J4.3, U6.23 (~{DCD}), U6.24 (~{CTS})
- no-connect marks 26 -> 24
